Commit message: 2 drone spawning + surface outline

File: src/drone/urdf/drone2.xacro (robot description, xacro)
@@ -1,4 +1,4 @@
 <?xml version='1.0'?>
-<robot name="drone" xmlns:xacro="http://www.ros.org/wiki/xacro">
+<robot name="drone2" xmlns:xacro="http://www.ros.org/wiki/xacro">
   <!-- ===== Properties ===== -->
   <xacro:property name="camera_width" value="0.02"/>
@@ -8,9 +8,9 @@
   <xacro:property name="depth_cam_mass" value="0.01"/>
   <xacro:property name="depth_cam_size" value="0.03"/>
-  <xacro:property name="chassis_mass" value="19"/>
+  <xacro:property name="chassis_mass" value="2"/>
   <xacro:property name="chassis_collision_x" value="0.20"/>
   <xacro:property name="chassis_collision_y" value="0.20"/>
-  <xacro:property name="chassis_collision_z_top" value="0.05"/>
-  <xacro:property name="chassis_collision_z_bottom" value="0.05"/>
+  <xacro:property name="chassis_collision_z_top" value="0.07442"/>
+  <xacro:property name="chassis_collision_z_bottom" value="0.02361"/>
   <xacro:include filename="$(find drone)/urdf/macros.xacro"/>
   <xacro:include filename="$(find drone)/urdf/materials.xacro"/>
@@ -82,5 +82,5 @@
     <parent link="chassis"/>
     <child link="camera_link"/>
-    <origin xyz="0 0 0" rpy="0 1.5708 0"/>
+    <origin xyz="0 0 0" rpy="0 0 0"/>
   </joint>
   <gazebo reference="camera_link">
@@ -91,6 +91,6 @@
       <horizontal_fov>0.65</horizontal_fov>
       <image>
-        <width>1400</width>
-        <height>650</height>
+        <width>1920</width>
+        <height>1080</height>
         <format>R8G8B8</format>
       </image>
@@ -101,8 +101,8 @@
     </camera>
     <plugin name="gazebo_ros_camera" filename="libgazebo_ros_camera.so">
-      <robotNamespace>/D1</robotNamespace>
+      <robotNamespace>/D2</robotNamespace>
       <cameraName>rgb_camera</cameraName>
       <frameName>rgb_camera_link</frameName>
-      <updateRate>60</updateRate>
+      <updateRate>30</updateRate>
     </plugin>
   </sensor>
@@ -166,10 +166,10 @@
     <sensor type="depth" name="depth_camera_sensor">
       <always_on>true</always_on>
-      <update_rate>150</update_rate>
+      <update_rate>200</update_rate>
       <camera>
-        <horizontal_fov>1.1</horizontal_fov>
+        <horizontal_fov>1</horizontal_fov>
         <image>
-          <width>300</width>
-          <height>150</height>
+          <width>650</width>
+          <height>300</height>
           <format>L8</format>
         </image>
@@ -180,11 +180,17 @@
       </camera>
       <plugin name="gazebo_ros_depth_camera" filename="libgazebo_ros_depth_camera.so">
-        <camera_name>D1/depth_camera</camera_name>
+        <camera_name>D2/depth_camera</camera_name>
         <frame_name>depth_camera_link</frame_name>
-        <update_rate>120</update_rate>
-        <robotNamespace>/D1</robotNamespace>
+        <update_rate>200</update_rate>
+        <robotNamespace>/D2</robotNamespace>
       </plugin>
     </sensor>
   </gazebo>
+  <gazebo reference="back_link">
+    <material>Gazebo/Red</material>
+  </gazebo>
+  <gazebo reference="front_link">
+    <material>Gazebo/Blue</material>
+  </gazebo>
   <!--============================================================================-->
   <!--                           DRONE CONTROL PLUGIN                             -->
@@ -192,5 +198,5 @@
   <gazebo>
     <plugin name="drone_control" filename="libSimpleBodyDroneControlPlugin.so">
-      <namespace>D1</namespace>
+      <namespace>D2</namespace>
     </plugin>
   </gazebo>

File: src/drone/urdf/materials.xacro (robot description, xacro)
@@ -5,5 +5,5 @@
 	</material>
 	<material name="blue">
-	  <color rgba="0.0 0.0 0.8 1.0"/>
+	  <color rgba="0.0 0.0 0.1 1.0"/>
 	</material>
 	<material name="green">
@@ -20,5 +20,5 @@
 	</material>
 	<material name="red">
-	  <color rgba="0.8 0.0 0.0 1.0"/>
+	  <color rgba="0.1 0.0 0.0 1.0"/>
 	</material>
 	<material name="white">
