Commit message: more files

File: src/drone/urdf/drone.xacro (robot description, xacro)
@@ -89,7 +89,7 @@
     <update_rate>120</update_rate>
     <camera>
-      <horizontal_fov>0.65</horizontal_fov>
+      <horizontal_fov>0.6</horizontal_fov>
       <image>
-        <width>1400</width>
+        <width>1500</width>
         <height>650</height>
         <format>R8G8B8</format>
@@ -104,5 +104,5 @@
       <cameraName>rgb_camera</cameraName>
       <frameName>rgb_camera_link</frameName>
-      <updateRate>60</updateRate>
+      <updateRate>165</updateRate>
     </plugin>
   </sensor>

File: src/drone/urdf/drone2.xacro (robot description, xacro)
@@ -8,9 +8,9 @@
   <xacro:property name="depth_cam_mass" value="0.01"/>
   <xacro:property name="depth_cam_size" value="0.03"/>
-  <xacro:property name="chassis_mass" value="2"/>
+  <xacro:property name="chassis_mass" value="19"/>
   <xacro:property name="chassis_collision_x" value="0.20"/>
   <xacro:property name="chassis_collision_y" value="0.20"/>
-  <xacro:property name="chassis_collision_z_top" value="0.07442"/>
-  <xacro:property name="chassis_collision_z_bottom" value="0.02361"/>
+  <xacro:property name="chassis_collision_z_top" value="0.05"/>
+  <xacro:property name="chassis_collision_z_bottom" value="0.05"/>
   <xacro:include filename="$(find drone)/urdf/macros.xacro"/>
   <xacro:include filename="$(find drone)/urdf/materials.xacro"/>
@@ -82,5 +82,5 @@
     <parent link="chassis"/>
     <child link="camera_link"/>
-    <origin xyz="0 0 0" rpy="0 0 0"/>
+    <origin xyz="0 0 0" rpy="0 1.5708 0"/>
   </joint>
   <gazebo reference="camera_link">
@@ -89,8 +89,8 @@
     <update_rate>120</update_rate>
     <camera>
-      <horizontal_fov>0.65</horizontal_fov>
+      <horizontal_fov>0.6</horizontal_fov>
       <image>
-        <width>1920</width>
-        <height>1080</height>
+        <width>1500</width>
+        <height>650</height>
         <format>R8G8B8</format>
       </image>
@@ -104,5 +104,5 @@
       <cameraName>rgb_camera</cameraName>
       <frameName>rgb_camera_link</frameName>
-      <updateRate>30</updateRate>
+      <updateRate>60</updateRate>
     </plugin>
   </sensor>
@@ -166,10 +166,10 @@
     <sensor type="depth" name="depth_camera_sensor">
       <always_on>true</always_on>
-      <update_rate>200</update_rate>
+      <update_rate>150</update_rate>
       <camera>
-        <horizontal_fov>1</horizontal_fov>
+        <horizontal_fov>1.1</horizontal_fov>
         <image>
-          <width>650</width>
-          <height>300</height>
+          <width>300</width>
+          <height>150</height>
           <format>L8</format>
         </image>
@@ -182,14 +182,8 @@
         <camera_name>D2/depth_camera</camera_name>
         <frame_name>depth_camera_link</frame_name>
-        <update_rate>200</update_rate>
+        <update_rate>120</update_rate>
         <robotNamespace>/D2</robotNamespace>
       </plugin>
     </sensor>
-  </gazebo>
-  <gazebo reference="back_link">
-    <material>Gazebo/Red</material>
-  </gazebo>
-  <gazebo reference="front_link">
-    <material>Gazebo/Blue</material>
   </gazebo>
   <!--============================================================================-->

Commit message: working competition sign cycle

File: src/drone/urdf/drone.xacro (robot description, xacro)
@@ -178,5 +178,5 @@
         <camera_name>D1/depth_camera</camera_name>
         <frame_name>depth_camera_link</frame_name>
-        <update_rate>120</update_rate>
+        <update_rate>250</update_rate>
         <robotNamespace>/D1</robotNamespace>
       </plugin>

File: src/drone/urdf/drone2.xacro (robot description, xacro)
@@ -9,6 +9,6 @@
   <xacro:property name="depth_cam_size" value="0.03"/>
   <xacro:property name="chassis_mass" value="19"/>
-  <xacro:property name="chassis_collision_x" value="0.20"/>
-  <xacro:property name="chassis_collision_y" value="0.20"/>
+  <xacro:property name="chassis_collision_x" value="0.15"/>
+  <xacro:property name="chassis_collision_y" value="0.15"/>
   <xacro:property name="chassis_collision_z_top" value="0.05"/>
   <xacro:property name="chassis_collision_z_bottom" value="0.05"/>
@@ -168,5 +168,5 @@
       <update_rate>150</update_rate>
       <camera>
-        <horizontal_fov>1.1</horizontal_fov>
+        <horizontal_fov>0.3</horizontal_fov>
         <image>
           <width>300</width>
