Commit message: images

File: src/2025_competition/robbie/urdf/robbie.xacro (robot description, xacro)
@@ -105,4 +105,18 @@
     </visual>
   </link>
+  <link name='camera_linkRead'>
+    <xacro:box_inertial name="camera_linkRead" m="${camera_mass}" x="${camera_width}" y="${camera_length}" z="${camera_height}"/>
+    <collision name='camera_link_collision'>
+      <geometry>
+        <box size="${camera_length} ${camera_width} ${camera_height}"/>
+      </geometry>
+    </collision>
+    <visual name='camera_link_visual'>
+      <origin xyz="0 0 0" rpy=" 0 0 0"/>
+      <geometry>
+        <box size="${camera_length} ${camera_width} ${camera_height}"/>
+      </geometry>
+    </visual>
+  </link>
   <joint name="wheel_FR_joint" type="continuous">
     <parent link="chassis"/>
@@ -137,4 +151,9 @@
     <child link="camera_link"/>
     <origin xyz="${chassis_length/2} 0 ${chassis_height/2+camera_height/2}"/>
+  </joint>
+  <joint name="cameraRead_joint" type="fixed">
+    <parent link="camera_link"/>
+    <child link="camera_linkRead"/>
+    <origin xyz="0 0 ${camera_height/2}"/>
   </joint>
   <gazebo reference="chassis">
@@ -177,6 +196,6 @@
         <horizontal_fov>1.75</horizontal_fov>
         <image>
-          <width>3840</width>
-          <height>2160</height>
+          <width>800</width>
+          <height>800</height>
           <format>R8G8B8</format>
         </image>
@@ -210,3 +229,42 @@
     </sensor>
   </gazebo>
+ <gazebo reference="camera_linkRead">
+    <sensor type="camera" name="camera2">
+      <update_rate>30.0</update_rate>
+      <camera name="head">
+        <horizontal_fov>1.75</horizontal_fov>
+        <image>
+          <width>2160</width>
+          <height>2160</height>
+          <format>R8G8B8</format>
+        </image>
+        <clip>
+          <near>0.02</near>
+          <far>300</far>
+        </clip>
+        <noise>
+          <type>gaussian</type>
+          <!-- Noise is sampled independently per pixel on each frame.
+              That pixel's noise value is added to each of its color
+              channels, which at that point lie in the range [0,1]. -->
+          <mean>0.0</mean>
+          <stddev>0.007</stddev>
+        </noise>
+      </camera>
+      <plugin name="camera_controller" filename="libgazebo_ros_camera.so">
+        <alwaysOn>true</alwaysOn>
+        <updateRate>0.0</updateRate>
+        <cameraName>rrbot/camera2</cameraName>
+        <imageTopicName>image_raw</imageTopicName>
+        <cameraInfoTopicName>camera_info</cameraInfoTopicName>
+        <frameName>camera_linkRead</frameName>
+        <hackBaseline>0.07</hackBaseline>
+        <distortionK1>0.0</distortionK1>
+        <distortionK2>0.0</distortionK2>
+        <distortionK3>0.0</distortionK3>
+        <distortionT1>0.0</distortionT1>
+        <distortionT2>0.0</distortionT2>
+      </plugin>
+    </sensor>
+  </gazebo>
 </robot>

Commit message: temp save

File: src/2025_competition/robbie/urdf/robbie.xacro (robot description, xacro)
@@ -105,4 +105,18 @@
     </visual>
   </link>
+  <link name='camera_linkRead'>
+    <xacro:box_inertial name="camera_linkRead" m="${camera_mass}" x="${camera_width}" y="${camera_length}" z="${camera_height}"/>
+    <collision name='camera_link_collision'>
+      <geometry>
+        <box size="${camera_length} ${camera_width} ${camera_height}"/>
+      </geometry>
+    </collision>
+    <visual name='camera_link_visual'>
+      <origin xyz="0 0 0" rpy=" 0 0 0"/>
+      <geometry>
+        <box size="${camera_length} ${camera_width} ${camera_height}"/>
+      </geometry>
+    </visual>
+  </link>
   <joint name="wheel_FR_joint" type="continuous">
     <parent link="chassis"/>
@@ -137,4 +151,9 @@
     <child link="camera_link"/>
     <origin xyz="${chassis_length/2} 0 ${chassis_height/2+camera_height/2}"/>
+  </joint>
+  <joint name="cameraRead_joint" type="fixed">
+    <parent link="camera_link"/>
+    <child link="camera_linkRead"/>
+    <origin xyz="0 0 ${camera_height/2}"/>
   </joint>
   <gazebo reference="chassis">
@@ -175,5 +194,5 @@
       <update_rate>30.0</update_rate>
       <camera name="head">
-        <horizontal_fov>1.3962634</horizontal_fov>
+        <horizontal_fov>2</horizontal_fov>
         <image>
           <width>800</width>
@@ -210,3 +229,47 @@
     </sensor>
   </gazebo>
+ <gazebo reference="camera_linkRead">
+    <sensor type="camera" name="camera2">
+      <update_rate>30.0</update_rate>
+      <camera name="head">
+        <horizontal_fov>1.75</horizontal_fov>
+        <image>
+          <width>2160</width>
+          <height>2160</height>
+          <format>R8G8B8</format>
+        </image>
+        <clip>
+          <near>0.02</near>
+          <far>300</far>
+        </clip>
+        <noise>
+          <type>gaussian</type>
+          <!-- Noise is sampled independently per pixel on each frame.
+              That pixel's noise value is added to each of its color
+              channels, which at that point lie in the range [0,1]. -->
+          <mean>0.0</mean>
+          <stddev>0.007</stddev>
+        </noise>
+      </camera>
+      <plugin name="camera_controller" filename="libgazebo_ros_camera.so">
+        <alwaysOn>true</alwaysOn>
+        <updateRate>0.0</updateRate>
+        <cameraName>rrbot/camera2</cameraName>
+        <imageTopicName>image_raw</imageTopicName>
+        <cameraInfoTopicName>camera_info</cameraInfoTopicName>
+        <frameName>camera_linkRead</frameName>
+        <hackBaseline>0.07</hackBaseline>
+        <distortionK1>0.0</distortionK1>
+        <distortionK2>0.0</distortionK2>
+        <distortionK3>0.0</distortionK3>
+        <distortionT1>0.0</distortionT1>
+        <distortionT2>0.0</distortionT2>
+      </plugin>
+    </sensor>
+  </gazebo>
+  <gazebo>
+    <plugin name="clueboard_handler" filename="libClueboardHandler.so">
+      <namespace>R1</namespace>
+    </plugin>
+  </gazebo>
 </robot>

File: src/drone/urdf/drone.xacro (robot description, xacro)
@@ -38,8 +38,8 @@
   </link>
   <!--============================================================================-->
-  <!--                         FRONT + BACK LINKS                                 -->
+  <!--                         FRONT + BACK LINKS (visual only)                   -->
   <!--============================================================================-->
   <link name="back_link">
-    <xacro:sphere_inertial name="back_link" m="0.5" r="0.05"/>
+    <xacro:sphere_inertial name="back_link" m="0.01" r="0.05"/>
     <visual name="back_visual">
       <geometry>
@@ -49,5 +49,5 @@
   </link>
   <link name="front_link">
-    <xacro:sphere_inertial name="front_link" m="0.5" r="0.05"/>
+    <xacro:sphere_inertial name="front_link" m="0.01" r="0.05"/>
     <visual name="front_visual">
       <geometry>
@@ -85,27 +85,27 @@
   </joint>
   <gazebo reference="camera_link">
-  <sensor type="camera" name="rgb_camera_sensor">
-    <always_on>true</always_on>
-    <update_rate>120</update_rate>
-    <camera>
-      <horizontal_fov>0.6</horizontal_fov>
-      <image>
-        <width>1500</width>
-        <height>650</height>
-        <format>R8G8B8</format>
-      </image>
-      <clip>
-        <near>0.05</near>
-        <far>50.0</far>
-      </clip>
-    </camera>
-    <plugin name="gazebo_ros_camera" filename="libgazebo_ros_camera.so">
-      <robotNamespace>/D1</robotNamespace>
-      <cameraName>rgb_camera</cameraName>
-      <frameName>rgb_camera_link</frameName>
-      <updateRate>165</updateRate>
-    </plugin>
-  </sensor>
-</gazebo>
+    <sensor type="camera" name="rgb_camera_sensor">
+      <always_on>true</always_on>
+      <update_rate>120</update_rate>
+      <camera>
+        <horizontal_fov>0.6</horizontal_fov>
+        <image>
+          <width>1500</width>
+          <height>650</height>
+          <format>R8G8B8</format>
+        </image>
+        <clip>
+          <near>0.05</near>
+          <far>50.0</far>
+        </clip>
+      </camera>
+      <plugin name="gazebo_ros_camera" filename="libgazebo_ros_camera.so">
+        <robotNamespace>/D1</robotNamespace>
+        <cameraName>rgb_camera</cameraName>
+        <frameName>rgb_camera_link</frameName>
+        <updateRate>165</updateRate>
+      </plugin>
+    </sensor>
+  </gazebo>
   <!--============================================================================-->
   <!--                                  IMU                                       -->
@@ -153,14 +153,10 @@
     </visual>
   </link>
-  <!-- Mount it under the chassis -->
   <joint name="depth_camera_mount" type="fixed">
     <parent link="chassis"/>
     <child link="depth_camera_link"/>
-    <!-- Point DOWNWARD: rpy = -90deg roll -->
+    <!-- Point downward -->
     <origin xyz="0 0 0" rpy="0 1.5708 0"/>
   </joint>
-  <!--=======================-->
-  <!--  SENSOR ON THE LINK   -->
-  <!--=======================-->
   <gazebo reference="depth_camera_link">
     <sensor type="depth" name="depth_camera_sensor">
@@ -194,4 +190,5 @@
       <namespace>D1</namespace>
     </plugin>
+    <enable_wind>true</enable_wind>
   </gazebo>
 </robot>

File: src/drone/urdf/drone2.xacro (robot description, xacro)
@@ -82,15 +82,15 @@
     <parent link="chassis"/>
     <child link="camera_link"/>
-    <origin xyz="0 0 0" rpy="0 1.5708 0"/>
+    <origin xyz="0 0 0" rpy="0 0 0"/>
   </joint>
   <gazebo reference="camera_link">
   <sensor type="camera" name="rgb_camera_sensor">
     <always_on>true</always_on>
-    <update_rate>120</update_rate>
+    <update_rate>30</update_rate>
     <camera>
-      <horizontal_fov>0.6</horizontal_fov>
+      <horizontal_fov>1.75</horizontal_fov>
       <image>
-        <width>1500</width>
-        <height>650</height>
+        <width>1800</width>
+        <height>1200</height>
         <format>R8G8B8</format>
       </image>
@@ -132,5 +132,5 @@
         <topicName>imu/data</topicName>
         <frameName>imu_link</frameName>
-        <updateRateHZ>144</updateRateHZ>
+        <updateRateHZ>250</updateRateHZ>
       </plugin>
     </sensor>
@@ -194,4 +194,5 @@
       <namespace>D2</namespace>
     </plugin>
+    <enable_wind>true</enable_wind>
   </gazebo>
 </robot>
